Commit message: comment collision shape avoiding object drop

File: src/magma_scenarios/envs/laundry/washmachine-103781/mobility.urdf (robot description, URDF)
Before this commit: robot partnet_ae8441235538d4415d85df7c37878bb6, 7 links, 6 joints
Links:
- link link_5: geometry collision mesh filename=textured_objs/original-12.obj; collision mesh filename=textured_objs/original-2.obj
