Commit message: fix the cardboard box collision to follow mesh

File: src/magma_scenarios/assets/box-100154/mobility.urdf (robot description, URDF)
Before this commit: robot partnet_33b1e78a6d49c2d67aa983983f9bf36, 6 links, 5 joints
Links:
- link link_4: geometry collision mesh filename=textured_objs/original-3.obj; collision mesh filename=textured_objs/original-4.obj
